File: Rev B/component_tester_adapter.kicad_pcb (KiCad board)
At the start: 2 copper layers, 72 x 75 mm, 27 parts, among them J1 microUSB, J2 LiPo, J3 9V, Q1 BC847, Q2 BC847, SW1 power, U1 MCP73831, U2 MCP1661

Commit message: added REV B
Parts:
- added REF**: OSHW-Logo_5.7x6mm_SilkScreen, Symbol:OSHW-Logo_5.7x6mm_SilkScreen, B.Cu at (184.2, 97.2)
